File: HeatIndex/HeatIndex.kicad_pcb (KiCad board)
At the start: 4 copper layers, 95 x 78 mm, 94 parts, among them J2 Conn_01x04_Socket, J6 Screw_Terminal_01x16, J7 Screw_Terminal_01x16, K1 SRD-05VDC-SL-C, K2 SRD-05VDC-SL-C, K3 SRD-05VDC-SL-C, K4 SRD-05VDC-SL-C, Q3 Q_NMOS_Depletion_GSD, Q4 Q_NMOS_Depletion_GSD, Q5 Q_NMOS_Depletion_GSD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

Commit message: -push firmware
Other:
- board text added: "1"
Changed lines of the file:
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@@
 		(tags "resistor handsolder")
 		(property "Reference" "R32"
-			(at 0.04 1.55 0)
+			(at -0.69 0.5 0)
 			(layer "F.SilkS")
 			(effects
@@
 		)
 		(property "Value" "1k"
-			(at 0 1.43 0)
+			(at -0.73 0.38 0)
 			(layer "F.Fab")
 			(effects
@@
 		)
 	)
+	(gr_text "1"
+		(at 60.2 109.6025 0)
+		(layer "B.SilkS")
+		(effects
+			(font
+				(size 1 1)
+				(thickness 0.15)
+			)
+			(justify mirror)
+		)
+	)
+	(gr_text "1"
+		(at 52.6 103.6 0)
+		(layer "B.SilkS")
+		(effects
+			(font
+				(size 1 1)
+				(thickness 0.15)
+			)
+			(justify mirror)
+		)
+	)
+	(gr_text "1"
+		(at 53.4 109.6 0)
+		(layer "B.SilkS")
+		(effects
+			(font
+				(size 1 1)
+				(thickness 0.15)
+			)
+			(justify mirror)
+		)
+	)
+	(gr_text "1"
+		(at 60.2 105 0)
+		(layer "B.SilkS")
+		(effects
+			(font
+				(size 1 1)
+				(thickness 0.15)
+			)
+			(justify mirror)
+		)
+	)
