File: HeatIndex/HeatIndex.kicad_sch (KiCad schematic)
At the start: 94 parts, among them J2 Conn_01x04_Socket, J6 Screw_Terminal_01x16, J7 Screw_Terminal_01x16, K1 SRD-05VDC-SL-C, K2 SRD-05VDC-SL-C, K3 SRD-05VDC-SL-C, K4 SRD-05VDC-SL-C, Q3 Q_NMOS_Depletion_GSD, Q4 Q_NMOS_Depletion_GSD, Q5 Q_NMOS_Depletion_GSD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

Commit message: -push firmware
Changed lines of the file:
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@@
 	(generator_version "9.0")
 	(paper "A2")
+	(rectangle
+		(start 242.57 228.6)
+		(end 317.5 308.61)
+		(stroke
+			(width 0)
+			(type default)
+		)
+		(fill
+			(type none)
+		)
+	)
+	(rectangle
+		(start 433.07 53.34)
+		(end 572.77 265.43)
+		(stroke
+			(width 0)
+			(type default)
+		)
+		(fill
+			(type none)
+		)
+	)
+	(rectangle
+		(start 245.11 320.04)
+		(end 337.82 394.97)
+		(stroke
+			(width 0)
+			(type default)
+		)
+		(fill
+			(type none)
+		)
+	)
+	(rectangle
+		(start 215.9 93.98)
+		(end 354.33 215.9)
+		(stroke
+			(width 0)
+			(type default)
+		)
+		(fill
+			(type none)
+		)
+	)
+	(rectangle
+		(start 203.2 10.16)
+		(end 365.76 82.55)
+		(stroke
+			(width 0)
+			(type default)
+		)
+		(fill
+			(type none)
+		)
+	)
 	(text "RELAY1\n"
 		(exclude_from_sim no)
